File: NER22A/NER22A.kicad_sch (KiCad schematic)
At the start: 0 parts

Commit message: Added accumulator organization
Other:
- added sheet Accumulator 1 (accumulator1.kicad_sch)
- added sheet Accumulator 2 (accumulator2.kicad_sch)
Changed lines of the file:
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@@
 (kicad_sch (version 20211123) (generator eeschema)
-  (paper "A1")
+  (paper "A2")
   (title_block
     (title "NER22A Master Schematic")
@@
     (company "Northeastern Electric Racing")
   )
+  (sheet (at 80.01 64.77) (size 85.09 82.55) (fields_autoplaced)
+    (stroke (width 0.1524) (type solid) (color 0 0 0 0))
+    (fill (color 0 0 0 0.0000))
+    (property "Sheet name" "Accumulator 1" (id 0) (at 80.01 64.0584 0)
+      (effects (font (size 1.27 1.27)) (justify left bottom))
+    )
+    (property "Sheet file" "accumulator1.kicad_sch" (id 1) (at 80.01 147.9046 0)
+      (effects (font (size 1.27 1.27)) (justify left top))
+    )
+  )
+  (sheet (at 180.34 64.77) (size 91.44 82.55) (fields_autoplaced)
+    (stroke (width 0.1524) (type solid) (color 0 0 0 0))
+    (fill (color 0 0 0 0.0000))
+    (property "Sheet name" "Accumulator 2" (id 0) (at 180.34 64.0584 0)
+      (effects (font (size 1.27 1.27)) (justify left bottom))
+    )
+    (property "Sheet file" "accumulator2.kicad_sch" (id 1) (at 180.34 147.9046 0)
+      (effects (font (size 1.27 1.27)) (justify left top))
+    )
+  )
   (sheet_instances
     (path "/" (page "1"))
+    (path "/2b9f2be9-94ac-4f24-8583-0445b8833796" (page "2"))
+    (path "/2b9f2be9-94ac-4f24-8583-0445b8833796/f6569233-c48b-4db8-951d-35f69f8f9cea" (page "3"))
+    (path "/2b9f2be9-94ac-4f24-8583-0445b8833796/8e3a6f27-2c9d-4cd9-aa19-4d4f86271d71" (page "4"))
+    (path "/2b9f2be9-94ac-4f24-8583-0445b8833796/43c1c9f2-aa3d-4906-bafc-86f432ad610b" (page "5"))
+    (path "/f0a6d14d-7d1c-42e4-8256-766a74ad9e63" (page "6"))
+    (path "/f0a6d14d-7d1c-42e4-8256-766a74ad9e63/a6be1d04-711b-420d-9ef0-f8c48519c795" (page "7"))
+    (path "/f0a6d14d-7d1c-42e4-8256-766a74ad9e63/691a96d4-55b0-4fa9-8a90-ccbdbbcfafed" (page "8"))
+    (path "/f0a6d14d-7d1c-42e4-8256-766a74ad9e63/4b85252a-2f82-4b70-9d64-a194fd6a4bd1" (page "9"))
   )
 )

Commit message: Tractive system schematic
Parts:
- added D? (x2): LED, symbol Device:LED
- added F? (x9): 1A, symbol Device:Fuse
- added F?: TS Fuse, symbol Device:Fuse
- added K? (x2): AIR+, Relay_THT:Relay_1P1T_NO_10x24x18.8mm_Panasonic_ADW11xxxxW_THT, symbol Relay:ADW11
- added K? (x2): Discharge, Relay_THT:Relay_SPST_RAYEX-L90B, symbol Relay:RAYEX-L90B
- added K? (x2): AIR-, Relay_THT:Relay_1P1T_NO_10x24x18.8mm_Panasonic_ADW11xxxxW_THT, symbol Relay:ADW11
- added K?: Precharge, Relay_THT:Relay_1P1T_NO_10x24x18.8mm_Panasonic_ADW11xxxxW_THT, symbol Relay:ADW11
- added R? (x2): R, symbol Device:R
- added R? (x2): 15k, symbol Device:R
- added SW? (x4): SMD, symbol Switch:SW_DIP_x01
- added SW?: HVD, symbol Switch:SW_DIP_x01
- added U?: Energy_Meter, symbol NER:Energy_Meter
- added U?: TSMP, symbol NER:Conn2
- added U? (x2): TSAL_PCB, symbol NER:TSAL_PCB
- added U?: Bender_Isometer, symbol NER:Bender_Isometer
- added U?: SPPos-, symbol NER:Conn1
- added U?: SPNeg+, symbol NER:Conn1
- added U?: Emrax_228, symbol NER:Emrax_228
- added U?: SPNeg-, symbol NER:Conn1
- added U? (x2): TS Sense, symbol NER:Conn2
- added U? (x2): Conn8, symbol NER:Conn8
- added U?: Conn14, symbol NER:Conn14
- added U?: SPPos+, symbol NER:Conn1
- added U?: HV500, symbol NER:HV500
- added U?: Precharge_PCB, symbol NER:Precharge_PCB
Connections:
- new net: F?.2, U?. (TS-) (x4)
- new net: F?.1, U?. (TS-) (x4)
- new net: F?.2, U?. (TS-), U?. (TS-), U?.1
- new net: U?. (TS-), U?. (TS-), U?.1
- new net: K?.11A, K?.11B, K?.3, R?.1, U?. (TS-)
- new net: R?.2, U?.1
- new net: U?.2, U?.2 (x3)
- new net: D?.2 (A), U?. (TS-) (x2)
- new net: U?.1, U?.1 (x3)
- new net: F?.2, K?.3, R?.2, U?.1
- new net: F?.1, K?.12, K?.3, U?.1
- new net: U?. (Phase3), U?. (Res) (x3)
- new net: K?.1, U?. (SD+)
- new net: F?.1, F?.2, K?.12, K?.3, R?.1, U?. (SD+), U?.1
- new net: F?.2, K?.5, R?.1
- new net: K?.6, U?. (SD+)
- new net: K?.11A, K?.11B, R?.1
- new net: U?. (Phase3), U?.1 (x2)
- new net: F?.1, F?.2, SW?.2
- new net: U?.3, U?.3
- new net: U?.4, U?.4
- new net: U?.5, U?.5
- new net: U?.6, U?.6
- new net: U?.7, U?.7
- new net: K?.3, U?. (SD+)
- new net: K?.5, R?.2
- new net: F?.1, U?.1
- new net: R?.2, U?.2
- new net EM_Comm+: U?. (TS-), U?.5
- new net EM_Comm-: U?. (TS-), U?.6
- new net GLV: U?. (TS-), U?. (TS-), U?.1
- new net GND: D?.1 (K), D?.1 (K), K?.1, K?.1, K?.1, K?.1, K?.A2, K?.A2, U?. (SD+), U?. (TS-), U?. (TS-), U?. (TS-), U?. (TS-), U?.14
- new net IMD_Chas1: U?. (TS-), U?.7
- new net IMD_Chas2: U?. (TS-), U?.8
- new net IMD_Status: U?. (TS-), U?.9
- new net Segment 1/Seg+: SW?.1
- new net Segment 1/Seg-: F?.1, K?.5
- new net Segment 2/Seg+: SW?.1
- new net Segment 2/Seg-: SW?.2
- new net Segment 3/GLV_OUT: U?.1
- new net Segment 3/GND_OUT: U?.2
- new net Segment 3/Seg+: F?.2, K?.5
- new net Segment 3/Seg-: SW?.2
- new net Segment 3/isoIM_OUT: U?.4
- new net Segment 3/isoIP_OUT: U?.3
- new net Segment 4/GLV_IN: U?.1
- new net Segment 4/GND_IN: U?.2
- new net Segment 4/Seg+: SW?.1
- new net Segment 4/Seg-: F?.1, K?.5
- new net Segment 4/isoIM_IN: U?.4
- new net Segment 4/isoIP_IN: U?.3
- new net Segment 5/Seg+: SW?.1
- new net Segment 5/Seg-: SW?.2
- new net Segment 6/Seg+: SW?.1
- new net Segment 6/Seg-: SW?.2
- new net Shutdown: K?.6, K?.6, K?.6, K?.6, K?.A1, K?.A1, U?. (SD+), U?.2, U?.5, U?.5
- new net TSAL_High_Neg: U?. (TS-), U?.13
- new net TSAL_High_Pos: U?. (TS-), U?.11, U?.7, U?.7
- new net TSAL_Status_Neg: U?. (TS-), U?.12
- new net TSAL_Status_Pos: U?. (TS-), U?.10, U?.6, U?.6
- new net isoIM: U?.4
- new net isoIP: U?.3
- no-connect marks 0 -> 16
Other:
- removed sheet Accumulator 1
- removed sheet Accumulator 2
- added sheet Segment 1 (segment.kicad_sch)
- added sheet Segment 2 (segment.kicad_sch)
- added sheet Segment 3 (segment.kicad_sch)
- added sheet Segment 4 (segment.kicad_sch)
- added sheet Segment 5 (segment.kicad_sch)
- added sheet Segment 6 (segment.kicad_sch)
- note added: "Motor"
- note added: "Motor Controller"
- note added: "Negative Sidepod"
- note added: "Positive Sidepod"

Commit message: Changed some pin names
Connections:
- net Segment 3/GLV_OUT is gone; now on net Segment 3/12V_OUT: U?.1
- net TSAL_Status_Neg is gone; now on net TSAL_StatusNeg: U?. (TS-), U?.12
- net isoIM is gone; now on net SPI_IP_IN: U?.4
- net isoIP is gone; now on net SPI_IP_IN: U?.3
- net Shutdown: no longer K?.6, K?.6, K?.6, K?.6, K?.A1, K?.A1, U?. (SD+), U?.2, U?.5
- net TSAL_High_Pos: no longer U?. (TS-), U?.11
- net TSAL_Status_Pos: no longer U?. (TS-), U?.10
- net at U?.1: now also R?.2
- net at U?.2: now also U?.2
- net at U?.2: now also U?.2; no longer U?.2
- net at U?.1: now also F?.2, K?.3, R?.2; no longer U?.1
- net at U?. (Res): now also U?. (Phase3)
- net at U?. (Phase3): now also U?.1; no longer U?. (Res)
- net at U?.2: now also R?.2; no longer U?.2
- net Segment 3/12V_OUT: now reaches U?.1
- net Segment 3/12V_OUT: no longer U?.1
- net SD_12V: now reaches U?.5
- net SD_12V: now also K?.6, K?.6, K?.6, K?.6, K?.A1, K?.A1, U?. (SD+), U?.2; no longer U?.5
- net GLV_12V: now reaches U?.1
- net GLV_12V: now also U?. (TS-), U?. (TS-)
- net TSAL_StatusPos: now reaches U?.10
- net TSAL_StatusPos: now also U?. (TS-)
- net TSAL_HighPos: now reaches U?.11
- net TSAL_HighPos: now also U?. (TS-)
- net TSAL_StatusNeg: now reaches U?.12
- net TSAL_HighNeg: now reaches U?.13
- net TSAL_HighNeg: now also U?. (TS-)
- net SPI_IP_IN: now reaches U?.3
- removed net GLV: U?. (TS-), U?. (TS-), U?.1
- net Segment 4/GLV_IN renamed Segment 4/12V_IN
- removed net TSAL_High_Neg: U?. (TS-), U?.13
- new net: F?.2, U?. (TS-), U?. (TS-), U?.1
- new net: U?. (TS-), U?. (TS-), U?.1
- new net: U?.1, U?.1 (x2)
- new net: U?. (Phase3), U?. (Res) (x2)
- new net: U?.2, U?.2
- new net: U?.3, U?.3
- new net: U?.4, U?.4
- new net: U?.5, U?.5
- new net: U?.6, U?.6
- new net: U?.7, U?.7
Other:
- sheet Segment 1 ports: added 12V_IN, 12V_OUT; removed GLV_IN, GLV_OUT
- sheet Segment 2 ports: added 12V_IN, 12V_OUT; removed GLV_IN, GLV_OUT
- sheet Segment 3 ports: added 12V_IN, 12V_OUT; removed GLV_IN, GLV_OUT
- sheet Segment 4 ports: added 12V_IN, 12V_OUT; removed GLV_IN, GLV_OUT
- sheet Segment 5 ports: added 12V_IN, 12V_OUT; removed GLV_IN, GLV_OUT
- sheet Segment 6 ports: added 12V_IN, 12V_OUT; removed GLV_IN, GLV_OUT
- moved on the sheet: U?

Commit message: Changed
Parts:
- added R?: R, symbol Device:R
- U?: value Conn14 -> LV
Connections:
- net TSAL_Seg+_Pos: now reaches F?.2, U?. (TS-)
- net TSAL_Seg+_Pos: now also F?.1, U?. (TS-)
- net TSAL_Seg+_Neg: now reaches F?.1, U?. (TS-)
- net TSMP+: now reaches U?.1
- net TSMP+: now also R?.2, U?.2, U?.2
- net TSMP-: now reaches R?.2
- net TSMP-: now also U?.2; no longer U?.1
- net TSAL_Seg-_Pos: now reaches F?.2, U?. (TS-)
- net at U?.1: now also F?.2, K?.3, R?.2; no longer U?.1
- net at U?. (Res): now also U?. (Phase3)
- net at U?. (Phase3): now also U?.1; no longer U?. (Res)
- net at F?.1, F?.2, K?.12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: now also K?.3; no longer U?. (SD+)
- net IMD,EM_TS+: now reaches U?.1, U?.1
- net IMD,EM_TS+: now also F?.1
- net at U?.1: no longer U?.1
- net at U?.2: no longer U?.2
- removed net Segment 3/12V_OUT: U?.1
- removed net Segment 3/GND_OUT: U?.2
- net Segment 4/12V_IN: no longer names the net of U?.1
- net Segment 4/GND_IN: no longer names the net of U?.2
- new net: U?. (TS-), U?. (TS-)
- new net: U?. (TS-), U?. (TS-), U?.1
- new net: F?.2, K?.3, R?.1, R?.2, U?. (TS-)
- new net: U?.1, U?.1 (x2)
- new net: U?. (Phase3), U?. (Res) (x2)
- new net: K?.11A, K?.11B, R?.1
- new net: U?.2, U?.2
- new net: U?.3, U?.3
- new net: U?.4, U?.4
- new net: U?.5, U?.5
- new net: U?.6, U?.6
- new net: U?.7, U?.7
- no-connect marks 16 -> 14
Other:
- sheet Segment 1 ports: added none; removed 12V_IN, 12V_OUT, GND_IN, GND_OUT
- sheet Segment 2 ports: added none; removed 12V_IN, 12V_OUT, GND_IN, GND_OUT
- sheet Segment 3 ports: added none; removed 12V_IN, 12V_OUT, GND_IN, GND_OUT
- sheet Segment 4 ports: added none; removed 12V_IN, 12V_OUT, GND_IN, GND_OUT
- sheet Segment 5 ports: added none; removed 12V_IN, 12V_OUT, GND_IN, GND_OUT
- sheet Segment 6 ports: added none; removed 12V_IN, 12V_OUT, GND_IN, GND_OUT
- note added: "Charger"
- note added: "OFFBOARD"
- note added: "ONBOARD"
- note added: "Powertrain"
- note removed: "Motor"
- note removed: "Motor Controller"
- moved on the sheet: D?, F?, K?, R?, SW?, U?

Commit message: Made some changes
POg
Parts:
- removed F? (x4): 1A, symbol Device:Fuse
- removed U?: Bender_Isometer, symbol NER:Bender_Isometer
- added U?: Bender_Isometer, symbol NER:Bender_Isometer
Connections:
- net Shutdown is gone; now on net SD_12V: U?.5
- net TSAL_High_Pos is gone; now on net TSAL_RED: U?.7, U?.7
- net TSAL_Seg+_Neg is gone; now on net TSAL_RED: U?. (TS-)
- net TSAL_Seg+_Pos is gone; now on net TSAL_RED: U?. (TS-), U?. (TS-)
- net TSAL_Seg-_Pos is gone; now on net TSAL_RED: U?. (TS-)
- net TSAL_Status_Pos is gone; now on net TSAL_GRN: U?.6, U?.6
- net EM_Comm+: now also U?.3; no longer U?.5
- net EM_Comm-: now also U?.4; no longer U?.6
- net GLV_12V: now also U?. (TS-), U?. (TS-), U?.2, U?.2, U?. (TS-)
- net GND: now also U?. (TS-)
- net IMD_Chas1: now also U?.5, U?. (TS-); no longer U?.7
- net IMD_Chas2: now also U?.6, U?. (TS-); no longer U?.8
- net IMD_Status: now also U?.7, U?. (TS-); no longer U?.9
- net SPI_IM_IN: now also U?.11
- net SPI_IP_IN: now also U?.10; no longer U?.3, U?.4
- net TSMP+: no longer R?.2, U?.2
- net at U?.1: now also U?. (Phase3); no longer U?. (TS-)
- net at F?.2, K?.3, R?.1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: now also U?. (TS-)
- net at U?.1: now also F?.2, K?.3, R?.2; no longer U?.1
- net at U?. (Res): now also U?. (Phase3)
- net at U?. (Phase3): now also U?.1; no longer U?. (Res)
- net at U?.2: now also R?.2; no longer U?.2
- net TSAL_GRN: now reaches U?.6, U?.6
- net TSAL_GRN: now also U?. (TS-), U?. (TS-), U?.8
- net TSAL_RED: now reaches U?.7, U?.7
- net TSAL_RED: now also U?.9
- net IMD,EM_TS+: no longer names the net of F?.1, U?.1
- net IMD,EM_TS+: no longer U?.1
- removed net TSAL_HighNeg: U?. (TS-), U?.13
- removed net TSAL_HighPos: U?. (TS-), U?.11
- removed net TSAL_StatusNeg: U?. (TS-), U?.12
- removed net TSAL_StatusPos: U?. (TS-), U?.10
- new net: U?. (TS-), U?.1
- new net: U?. (TS-), U?. (TS-), U?.1
- new net: U?.1, U?.1
- new net: U?. (Phase3), U?. (Res) (x2)
- new net: U?.2, U?.2 (x2)
- new net: U?.3, U?.3
- new net: U?.4, U?.4
- new net: U?.5, U?.5
- new net: U?.6, U?.6
- new net: U?.7, U?.7
Other:
- moved on the sheet: D?, F?, R?

Commit message: Added charger
Parts:
- removed U? (x2): TS Sense, symbol NER:Conn2
- removed U? (x2): Conn8, symbol NER:Conn8
- removed U?: LV, symbol NER:Conn14
- added D?: AMS Fault, symbol Device:LED
- added D?: IMD Fault, symbol Device:LED
- added F? (x6): Fuse, symbol Device:Fuse
- added F? (x3): 1A, symbol Device:Fuse
- added J?: Conn_WallSocket_Earth, symbol Connector:Conn_WallSocket_Earth
- added K? (x2): Latching Relay, Relay_THT:Relay_DPDT_Schrack-RT2-FormC_RM5mm, symbol Relay:RT42xAxx
- added K?: Charger Safety, Relay_THT:Relay_SPST_RAYEX-L90B, symbol Relay:RAYEX-L90B
- added SW?: Charger Shutdown BRB, symbol Switch:SW_Push
- added SW?: IMD Reset, symbol Switch:SW_Push
- added SW?: AMS Reset, symbol Switch:SW_Push
- added U? (x2): Conn20, symbol NER:Conn20
- added U? (x2): Conn3, symbol NER:Conn3
- added U?: AC-DC, symbol NER:AC-DC
- added U?: HV, symbol NER:Conn2
- added U? (x2): Conn12, symbol NER:Conn12
- added U?: DC-DC, symbol NER:DC-DC
- added U?: Elcon_Charger, symbol NER:Elcon_Charger
- added U?: TSMP, symbol NER:Conn2
Connections:
- net EM_Comm+: now also U?.3, U?.3
- net EM_Comm-: now also U?.4, U?.4
- net GLV_12V: now also D?.2 (A), D?.2 (A), U?. (N), U?.1, U?.1, U?.1, U?.1
- net GND: now also J?.3 (EARTH), K?.11, K?.11, K?.A1, SW?.2, SW?.2, U?. (N), U?. (N), U?. (TS-), U?.10, U?.10, U?.11, U?.11, U?.12, U?.12, U?.20, U?.20
- net IMD_Chas1: now also U?.5, U?.5
- net IMD_Chas2: now also U?.6, U?.6
- net IMD_Status: now also K?.A2, U?.7, U?.7
- net SD_12V: now also U?.2, U?.2, U?.4, U?.4
- net SPI_IM_IN: now also U?.11
- net SPI_IP_IN: now also U?.10
- net Segment 3/isoIM_OUT: now also U?.3
- net Segment 3/isoIP_OUT: now also U?.2
- net Segment 4/isoIM_IN: now also U?.3
- net Segment 4/isoIP_IN: now also U?.2
- net TSAL_GRN: now also U?.5, U?.5, U?.8, U?.8
- net TSAL_RED: now also U?.6, U?.6, U?.9, U?.9
- net TSMP+: now also U?.1, U?.3
- net TSMP-: now also U?.2
- net at U?.1: now also U?. (Phase3), U?.2; no longer U?. (TS-)
- net at F?.2, K?.3, R?.1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: now also F?.2, F?.2; no longer U?. (TS-)
- net at U?.1: now also F?.2, K?.3, R?.2; no longer U?.1
- net at U?. (Res): now also U?. (Phase3)
- net at U?. (Phase3): now also U?.1, U?.1; no longer U?. (Res)
- net at F?.1, F?.2, K?.12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: now also F?.2
- net TS+_Sense: now reaches F?.1
- net TS+_Sense: now also U?.2
- net TSAL: now reaches R?.2
- net TSAL: now also U?.3
- new net: D?.1 (K), K?.12 (x2)
- new net: U?. (TS-), U?.1 (x2)
- new net: U?. (TS-), U?. (TS-), U?.2
- new net: U?.1, U?.1 (x3)
- new net: U?. (Phase3), U?. (Res) (x2)
- new net: U?.2, U?.2 (x2)
- new net: U?.3, U?.3 (x2)
- new net: F?.1, F?.1, K?.12
- new net: F?.2, U?. (N) (x2)
- new net: K?.14, K?.A1, SW?.1 (x2)
- new net: K?.21, K?.24
- new net: K?.24, SW?.1
- new net: F?.1, U?.1 (x2)
- new net: F?.2, J?.1 (AC_P)
- new net: F?.1, J?.2 (AC_N)
- new net: F?.1, U?. (TS-) (x2)
- new net: F?.1, U?. (N) (x2)
- new net: F?.2, F?.2, U?. (N)
- new net: F?.2, U?.2
- new net: U?.10, U?.10
- new net: U?.11, U?.11
- new net: U?.12, U?.12
- new net: U?.4, U?.4
- new net: U?.5, U?.5
- new net: U?.6, U?.6
- new net: U?.7, U?.7
- new net: U?.8, U?.8
- new net: U?.9, U?.9
- new net: K?.11A, K?.11B, U?. (N)
- new net: K?.A2, U?. (N)
- new net: SW?.2, U?. (N)
- new net 12V_DCDC: U?. (TS-), U?.14, U?.14, U?.7, U?.7
- new net AMS_Status: K?.A2
- new net CANH: U?. (N), U?. (TS-), U?.13, U?.13, U?.8, U?.8
- new net CANL: U?. (N), U?. (TS-), U?.12, U?.12, U?.9, U?.9
- new net CHRG_EN: K?.21
- new net SPI_IM: U?.11
- new net SPI_IP: U?.10
- no-connect marks 14 -> 13
Other:
- note added: "BMS"
- note added: "Charger Shutdown"
- note added: "HV"
- moved on the sheet: D?, F?, K?, R?, SW?, U?

Commit message: Updated wiring
Updated wiring based on wiring table in confluence
Parts:
- removed U?: TSMP, symbol NER:Conn2
- removed U?: TSAL_PCB, symbol NER:TSAL_PCB
- removed U? (x2): Conn3, symbol NER:Conn3
- removed U? (x2): Conn12, symbol NER:Conn12
- removed U?: Conn20, symbol NER:Conn20
- added F?: TS Fuse, symbol Device:Fuse
- added U1, U?: P2P LV, symbol NER:Conn8
- added U?: Charger, symbol NER:Conn6
- added U? (x2): P2P HV, symbol NER:Conn3
- added U?: ~, symbol NER:Shep_Controller22
- added U?: OrionCurrentSens, symbol NER:OrionCurrentSens
- added U?: DCDC Out, symbol NER:Conn2
- added U?: Vehicle LV, symbol NER:Conn6
- added U?: TSMP, symbol NER:Conn2
- added U?: Vehicle LV, symbol NER:Conn8
- added U?: TSAL_PCB, symbol NER:TSAL_PCB
Connections:
- net TSAL is gone; now on net TSMP+: R?.2
- net 12V_DCDC: no longer U?. (TS-)
- net CANH: no longer U?. (TS-)
- net CANL: no longer U?. (TS-)
- net EM_Comm+: no longer U?. (TS-)
- net EM_Comm-: no longer U?. (TS-)
- net GLV_12V: no longer U?. (TS-), U?. (TS-), U?. (TS-)
- net GND: now also U?.2 (TS-), U?.2 (TS-); no longer U?. (TS-), U?. (TS-), U?. (TS-), U?. (TS-)
- net IMD_Chas1: now also U?.3 (Ch1GND), U?.1; no longer U?. (TS-)
- net IMD_Chas2: now also U?.4 (Ch2GND), U?.2; no longer U?. (TS-)
- net IMD_Status: no longer U?. (TS-)
- net SD_12V: no longer K?.6, K?.6, K?.6, K?.6, K?.A1, K?.A1, U?. (SD+)
- net SPI_IM: now also U?.1 (Shutdown)
- net SPI_IP: now also U?.2 (IsoSPI_P)
- net Segment 3/Seg+: now also F?.1; no longer K?.5
- net Segment 3/isoIM_OUT: now also U?.1
- net Segment 3/isoIP_OUT: now also U?.2
- net Segment 4/isoIM_IN: now also U1.2
- net Segment 4/isoIP_IN: now also U1.3
- net TS+_Sense: now also U?.1
- net TSAL_GRN: no longer U?. (TS-)
- net TSAL_RED: no longer U?. (TS-)
- net TSMP+: now also U?.1, U?.3, U?.3
- net TSMP-: now also U?.2
- net at U?. (TS-): now also U?.2 (TS-); no longer U?.1
- net at D?.2 (A): now also U?.1 (TS+)
- net at F?.1: now also U?.2 (TS-)
- net at F?.2: now also U?.1 (TS+)
- net at U?.1: now also F?.2, K?.3, R?.2; no longer U?.1
- net at F?.2: now also U?.1 (TS+); no longer U?. (TS-)
- net at U?. (Res): now also U?. (Phase3)
- net at U?. (Phase3): now also U?.1, U?.1; no longer U?. (Res)
- net +TSAL PACK+: now reaches F?.2, K?.5, R?.1
- net +TSAL PACK+: now also U?.1 (TS+)
- net at SW?.2: now also U?.L1 (Load+); no longer F?.1
- net at F?.1: now also U?.2
- net at F?.1: now also U?.1 (TS-); no longer U?. (TS-)
- net at F?.1: now also U?.1 (TS+); no longer U?. (TS-)
- net at F?.1: now also U?.2 (TS-); no longer U?. (TS-)
- net at D?.2 (A): now also U?.1 (TS+); no longer U?. (TS-)
- net Segment 1/Seg- renamed -TSAL PACK-
- net -TSAL PACK-: now also U?.2 (TS-)
- net Segment 4/Seg- renamed +TSAL PACK-
- net +TSAL PACK-: now also U?.2 (TS-)
- new net: U?.1, U?.1 (Shutdown)
- new net: U?.2, U?.2 (IsoSPI_P)
- new net: U?.3, U?.3 (Shield)
- new net: U?.4, U?.4 (Current_Low)
- new net: U?.5, U?.5 (Interlock_24V)
- new net: U?.6, U?.6 (Interlock_Read)
- new net: U?.1, U?.1 (TS-)
- new net: U?.1, U?.1 (x2)
- new net: U?.2, U?.2
- new net: U?.3, U?.3
- new net: U?. (TS-), U?.1
- new net: U?.1 (GLV+), U?.1 (Shutdown)
- new net: U?.2 (GND), U?.2 (IsoSPI_P)
- new net: U?.3 (CANH), U?.3 (Shield)
- new net: U?.4 (CANL), U?.4 (Current_Low)
- new net: U?. (Phase3), U?. (Res) (x2)
- new net: F?.1, U?.L2 (Load-)
- new net: U?. (Phase3), U?.1, U?.2
- new net: U?.1, U?.1 (TS+)
- new net: U?.2, U?.2 (TS-) (x2)
- new net: U1.1, U?.1
- new net: U1.2, U?.2
- new net: U1.3, U?.3
- new net: U1.4, U?.4
- new net: U1.5, U?.5
- new net: U1.6, U?.6
- new net: U1.7, U?.7
- new net: U1.8, U?.8
- new net +Current_High: U1.7, U?.2(B) (C_High)
- new net +Current_Low: U1.6, U?.4(D) (C_Low)
- new net +Sensor_GND: U1.4, U?.3(C) (GND)
- new net +Sensor_Power: U1.5, U?.1(A) (+5_Pow)
- new net +TSAL_GND: U?.1 (TS+), U?.2 (TS-)
- new net +TSAL_GRN: U?.4 (Green), U?.5
- new net +TSAL_RED: U?.3 (Red), U?.4
- new net -TSAL PACK+: F?.2, K?.5, U?.1 (TS+)
- new net -TSAL_GND: U?.1 (TS+), U?.2 (IsoSPI_P)
- new net -TSAL_GRN: U?.4 (Green), U?.5
- new net -TSAL_RED: U?.3 (Red), U?.4
- new net Current_High: U?.5 (Interlock_24V), U?.7
- new net Current_Low: U?.4 (Current_Low), U?.6
- new net DCDC_CANH: U?.2, U?.2 (TS-)
- new net DCDC_CANL: U?.3, U?.3 (CANL)
- new net DCDC_GND: U?.1, U?.1 (TS+)
- new net GLV_24V: U?.3 (Shield), U?.8
- new net GLV_GND: U?.2 (IsoSPI_P), U?.6
- new net IMD_24V: U?.1 (Shutdown), U?.2 (TS-)
- new net IMD_Fault: U?.3, U?.8 (IMD_Fault)
- new net IMD_GND: U?.1 (TS-), U?.2 (IsoSPI_P)
- new net LV_Shutdown: U?.1 (Shutdown), U?.7
- new net SD_24V: K?.6, K?.6, K?.6, K?.6, K?.A1, K?.A1, U?. (SD+)
- new net SPI_Shield: U?.3 (Shield)
- new net Segment 3/isoISHIELD_OUT: U?.3
- new net Segment 4/isoISHIELD_IN: U1.1
- new net Sensor_GND: U?.1 (Shutdown), U?.4
- new net Sensor_Power: U?.3 (Shield), U?.5
- no-connect marks 13 -> 14
Other:
- sheet Segment 1 ports: added isoISHIELD_IN, isoISHIELD_OUT; removed none
- sheet Segment 2 ports: added isoISHIELD_IN, isoISHIELD_OUT; removed none
- sheet Segment 3 ports: added isoISHIELD_IN, isoISHIELD_OUT; removed none
- sheet Segment 4 ports: added isoISHIELD_IN, isoISHIELD_OUT; removed none
- sheet Segment 5 ports: added isoISHIELD_IN, isoISHIELD_OUT; removed none
- sheet Segment 6 ports: added isoISHIELD_IN, isoISHIELD_OUT; removed none
- moved on the sheet: D?, F?, K?, R?, SW?
