File: NER22A/NER22A.kicad_sch (KiCad schematic)
At the start: 66 parts

Commit message: Added LV Circuits
Added a first pass of all LV circuits to the Master Schematic. Also moved HV stuff into sub-sheets
Parts:
- removed D?: AMS Fault, symbol Device:LED
- removed D?: IMD Fault, symbol Device:LED
- removed D? (x2): LED, symbol Device:LED
- removed F? (x8): 1A, symbol Device:Fuse
- removed F? (x6): Fuse, symbol Device:Fuse
- removed F?: TS Fuse, symbol Device:Fuse
- removed J?: Conn_WallSocket_Earth, symbol Connector:Conn_WallSocket_Earth
- removed K? (x2): AIR+, Relay_THT:Relay_1P1T_NO_10x24x18.8mm_Panasonic_ADW11xxxxW_THT, symbol Relay:ADW11
- removed K? (x2): Latching Relay, Relay_THT:Relay_DPDT_Schrack-RT2-FormC_RM5mm, symbol Relay:RT42xAxx
- removed K? (x2): Discharge, Relay_THT:Relay_SPST_RAYEX-L90B, symbol Relay:RAYEX-L90B
- removed K? (x2): AIR-, Relay_THT:Relay_1P1T_NO_10x24x18.8mm_Panasonic_ADW11xxxxW_THT, symbol Relay:ADW11
- removed K?: Precharge, Relay_THT:Relay_1P1T_NO_10x24x18.8mm_Panasonic_ADW11xxxxW_THT, symbol Relay:ADW11
- removed K?: Charger Safety, Relay_THT:Relay_SPST_RAYEX-L90B, symbol Relay:RAYEX-L90B
- removed R? (x3): R, symbol Device:R
- removed R? (x2): 15k, symbol Device:R
- removed SW? (x4): SMD, symbol Switch:SW_DIP_x01
- removed SW?: HVD, symbol Switch:SW_DIP_x01
- removed SW?: Charger Shutdown BRB, symbol Switch:SW_Push
- removed SW?: IMD Reset, symbol Switch:SW_Push
- removed SW?: AMS Reset, symbol Switch:SW_Push
- removed U?: Energy_Meter, symbol NER:Energy_Meter
- removed U? (x2): Conn20, symbol NER:Conn20
- removed U? (x2): TSMP, symbol NER:Conn2
- removed U? (x2): TSAL_PCB, symbol NER:TSAL_PCB
- removed U?: SPPos-, symbol NER:Conn1
- removed U?: SPNeg+, symbol NER:Conn1
- removed U? (x2): Conn3, symbol NER:Conn3
- removed U?: SPNeg-, symbol NER:Conn1
- removed U?: Bender_Isometer, symbol NER:Bender_Isometer
- removed U?: AC-DC, symbol NER:AC-DC
- removed U?: HV, symbol NER:Conn2
- removed U? (x2): Conn12, symbol NER:Conn12
- removed U?: DC-DC, symbol NER:DC-DC
- removed U?: SPPos+, symbol NER:Conn1
- removed U?: Elcon_Charger, symbol NER:Elcon_Charger
- removed U?: Precharge_PCB, symbol NER:Precharge_PCB
- added -101 (x6), -103, -104, -105 (x2), -106 (x6), -107 (x3), -108 (x3), -109, -115, -2, -3: CHASSIS, symbol NER:CHASSIS
- added BT101 (x2): GLV Battery, symbol Device:Battery_Cell
- added D1: TSAL Dashboard Indicator, symbol Device:LED
- added D101: BRAKE_LIGHT, symbol NER:ST-R10_LED
- added D102 (x2): IMD Fault Indicator, symbol Device:LED
- added D102: BSPD Fault Indicator, symbol Device:LED
- added D103 (x2): BMS Fault Indicator, symbol Device:LED
- added D104: CAN Fault Indicator, symbol Device:LED
- added D104: MPU Fault Indicator, symbol Device:LED
- added D105: TSAL_150V_LED, symbol Device:LED
- added F1, F2, F3 (x2), F4, F5, F6, F7, F8, F9: 20A, symbol Device:Fuse
- added F10, F11, F12, F13: 7.5A, symbol Device:Fuse
- added J101 (x2): TS-, symbol Connector:Conn_01x01_Female
- added J102 (x2): TS+, symbol Connector:Conn_01x01_Female
- added J103 (x2): GND, symbol Connector:Conn_01x01_Female
- added LS101 (x2), LS102: Speaker, symbol Device:Speaker
- added M1 (x6), M101 (x6), M2 (x6): RadFan, symbol Motor:Fan
- added M10, M3, M4, M5, M6, M7, M8, M9: BattFan, symbol Motor:Fan_4pin
- added M103 (x2): Cooling Pump, symbol Motor:Motor_DC
- added R101: 3.01K, symbol Device:R
- added RV101, RV102, RV103, RV104: R_POT, symbol Device:R_POT
- added RV101: APPS2, symbol Device:R_POT
- added RV102: APPS1, symbol Device:R_POT
- added RV103: BSE2, symbol Device:R_POT
- added RV104: BSE1, symbol Device:R_POT
- added SW101 (x2): Brake Over-Travel Switch, symbol Switch:SW_SPST
- added SW102 (x2), SW103 (x2): Side BRB, symbol Switch:SW_Push_Open
- added SW105 (x2): Cockpit BRB, symbol Switch:SW_Push_Open
- added SW105: Inertia Switch, symbol Switch:SW_Push_Open
- added SW106 (x2): TSMS, symbol Switch:SW_SPST
- added SW107 (x2): TPST MOMENTARY BUTTON, symbol Switch:SW_DIP_x03
- added SW1A (x2), SW1B (x2): GLVMS, symbol Switch:SW_SPST
- added U101: RinehartPM100DX_MotorController, symbol NER:RinehartPM100DX_MotorController
Connections:
- net at U?. (Res): now also U?. (Phase3)
- net Accumulator/SPPos+: now reaches U?. (Phase3)
- net Accumulator/SPPos+: no longer U?. (Res)
- net LV_BOX/24V_Motor_Controller: now reaches U?.1 (12_Vin)
- new net: F3.1, SW1A.1 (A)
- new net: -105. (-), D102.1 (K), D103.1 (K), D104.1 (K)
- new net: -106. (-), M1.2 (-), M1.2 (-), M1.2 (-), M1.2 (-), M101.2 (-), M101.2 (-), M101.2 (-), M101.2 (-), M2.2 (-), M2.2 (-), M2.2 (-), M2.2 (-)
- new net: -115. (-), U101.6 (GND)
- new net: -106. (-), M1.2 (-), M101.2 (-), M2.2 (-) (x2)
- new net: F7.2, F8.2, F9.2, SW1B.2 (B)
- new net: -105. (-), D102.1 (K), D102.1 (K), D103.1 (K), D104.1 (K)
- new net: SW102.1 (A), SW103.1 (A) (x2)
- new net: -109. (-), D105.1 (K)
- new net: -103. (-), D101.3 (-)
- new net: U?. (Phase3), U?. (Res) (x2)
- new net: F1.1, F2.1, F3.1, SW1A.1 (A)
- new net: -108. (-), J103.1 (Pin_1), SW107.5, SW107.6
- new net: F10.2, M10.2 (+), M9.2 (+)
- new net: -107. (-), M103.2 (-) (x2)
- new net: F4.1, F5.1, F6.1, SW1A.2 (B)
- new net: F11.2, M7.2 (+), M8.2 (+)
- new net: SW105.2 (B), SW106.1 (A) (x2)
- new net: BT101.1 (+), F3.2
- new net: R101.1, U101.14 (XDCR_PWR)
- new net: R101.2, U101.24 (AIN2_Motor_Temp)
- new net: -108. (-), J103.1 (Pin_1), SW107.4, SW107.5, SW107.6
- new net: F12.2, M5.2 (+), M6.2 (+)
- new net: F13.2, M3.2 (+), M4.2 (+)
- new net: -2. (-), D1.1 (K)
- new net: SW105.1 (A), SW105.2 (B)
- new net Accumulator Container/DCDC_14.6V_1: SW1B.1 (A)
- new net Accumulator Container/DCDC_GND1: -3. (-)
- new net Accumulator Container/FanPWM: M10.4 (PWM), M3.4 (PWM), M4.4 (PWM), M5.4 (PWM), M6.4 (PWM), M7.4 (PWM), M8.4 (PWM), M9.4 (PWM)
- new net Accumulator Container/MC_AIR+: U101.7 (RLY2_Main)
- new net Accumulator Container/MC_Precharge+: U101.21 (RLY1_PreCharge)
- new net Accumulator Container/ShutdownLoop_GLV+: SW106.2 (B)
- new net Accumulator Container/TS+: U101.~ (TS-)
- new net Accumulator Container/TS-: U101.~ (TS-)
- new net Accumulator Container/TSAL_150V: D105.2 (A)
- new net Accumulator Container/TSAL_ACTIVE: D1.2 (A)
- new net Accumulator Container/TSMP+: J102.1 (Pin_1)
- new net Accumulator Container/TSMP-: J101.1 (Pin_1)
- new net Accumulator/24V_DCDC: SW1B.1 (A)
- new net Accumulator/IMD_Chas2: -106. (-)
- new net Accumulator/IMS_Chas1: -106. (-)
- new net Accumulator/SD_24V: SW106.2 (B)
- new net Accumulator/SPNeg-: U?. (Phase3)
- new net Accumulator/TSMP+: J102.1 (Pin_1)
- new net Accumulator/TSMP-: J101.1 (Pin_1)
- new net Brake_Light/GND: -106. (-)
- new net Dashboard/BRAKE1+: RV103.1
- new net Dashboard/BRAKE1-: RV103.3
- new net Dashboard/BRAKE1_INPUT: RV103.2
- new net Dashboard/BRAKE2+: RV104.1
- new net Dashboard/BRAKE2-: RV104.3
- new net Dashboard/BRAKE2_INPUT: RV104.2
- new net Dashboard/GND: -104. (-)
- new net Dashboard/GND: -107. (-)
- new net Dashboard/POT1+: RV101.1
- new net Dashboard/POT1-: RV101.3
- new net Dashboard/POT1_INPUT: RV101.2
- new net Dashboard/POT2+: RV102.1
- new net Dashboard/POT2-: RV102.3
- new net Dashboard/POT2_INPUT: RV102.2
- new net Dashboard/RTDS+: LS101.1
- new net Dashboard/RTDS-: LS101.2
- new net Dashboard/Speaker1+: LS101.1
- new net Dashboard/Speaker1-: LS101.2
- new net Dashboard/Speaker2+: LS102.1
- new net Dashboard/Speaker2-: LS102.2
- new net GLV Battery Board/BATT+: BT101.1 (+)
- new net GLV Battery Board/DCDC1: F7.1
- new net GLV Battery Board/DCDC2: F8.1
- new net GLV Battery Board/DCDC3: F9.1
- new net GLV Battery Board/GND: -101. (-), BT101.2 (-)
- new net GLV Battery Board/SYS1+: F1.2
- new net GLV Battery Board/SYS2+: F2.2
- new net GLV Battery Board/SYS3+: F3.2
- new net LV_BOX/12V_PUMP: M103.1 (+)
- new net LV_BOX/24V_BATTBOX_FAN1: M2.1 (+)
- new net LV_BOX/24V_BATTBOX_FAN10: M2.1 (+)
- new net LV_BOX/24V_BATTBOX_FAN11: M1.1 (+)
- new net LV_BOX/24V_BATTBOX_FAN12: M101.1 (+)
- new net LV_BOX/24V_BATTBOX_FAN2: M1.1 (+)
- new net LV_BOX/24V_BATTBOX_FAN3: M101.1 (+)
- new net LV_BOX/24V_BATTBOX_FAN4: M2.1 (+)
- new net LV_BOX/24V_BATTBOX_FAN5: M1.1 (+)
- new net LV_BOX/24V_BATTBOX_FAN6: M101.1 (+)
- new net LV_BOX/24V_BATTBOX_FAN7: M2.1 (+)
- new net LV_BOX/24V_BATTBOX_FAN8: M1.1 (+)
- new net LV_BOX/24V_BATTBOX_FAN9: M101.1 (+)
- new net LV_BOX/24V_BATTERY: SW1A.2 (B)
- new net LV_BOX/24V_DCDC: SW1B.2 (B)
- new net LV_BOX/24V_RADIATOR_FAN: M1.1 (+), M101.1 (+), M2.1 (+)
- new net LV_BOX/5V_Pedalbox_Sensors: RV101.1, RV102.1, RV103.1, RV104.1
- new net LV_BOX/APPS1: RV102.2
- new net LV_BOX/APPS2: RV101.2
- new net LV_BOX/BMS_INDICATOR: D103.2 (A)
- new net LV_BOX/BMS_RESET: SW107.2
- new net LV_BOX/BSE1: RV104.2
- new net LV_BOX/BSE2: RV103.2
- new net LV_BOX/BSPD_INDICATOR: D102.2 (A)
- new net LV_BOX/BSPD_RESET: SW107.3
- new net LV_BOX/GND_BATTERY: -101. (-), BT101.2 (-)
- new net LV_BOX/GND_Pedalbox_Sensors: RV101.3, RV102.3, RV103.3, RV104.3
- new net LV_BOX/IMD_INDICATOR: D102.2 (A)
- new net LV_BOX/IMD_RESET: SW107.1
- new net LV_BOX/MPU_INDICATOR: D104.2 (A)
- new net LV_BOX/SD_From_Side_BRBs: SW103.2 (B)
- new net LV_BOX/SD_To_Side_BRBs: SW102.2 (B)
- new net LV_BOX/Shutdown_From_BOTS: SW101.2 (B)
- new net LV_BOX/Shutdown_TO_BOTS: SW101.1 (A)
- new net LV_BOX/Shutdown_TO_COCKPIT_BRB: SW105.1 (A)
- new net Mechanical_Sensor_Board_1/GND: -101. (-)
- new net Mechanical_Sensor_Board_2/GND: -101. (-) (x2)
- new net Mechanical_Sensor_Board_3/GND: -101. (-)
- new net Power Distribution/12V_BattboxFansL1: F12.1
- new net Power Distribution/12V_BattboxFansL2: F13.1
- new net Power Distribution/12V_BattboxFansR1: F10.1
- new net Power Distribution/12V_BattboxFansR2: F11.1
- new net Power Distribution/12V_Brakelight: D101.1 (+), D101.2 (+)
- new net Power Distribution/12V_GLVMS1: F4.2
- new net Power Distribution/12V_GLVMS2: F5.2
- new net Power Distribution/12V_GLVMS3: F6.2
- new net Power Distribution/12V_MotorController: U101.8 (DIN2_Reverse)
- new net Power Distribution/12V_Pump: M103.1 (+)
- new net Power Distribution/12V_RadiatorFan: M1.1 (+), M101.1 (+), M2.1 (+)
- new net Power Distribution/BMS_Fault_Indicator: D103.2 (A)
- new net Power Distribution/BMS_Latch_Reset: SW107.2
- new net Power Distribution/CAN_Fault_Indicator: D104.2 (A)
- new net Power Distribution/GND_BattboxFansL1: M5.1 (-), M6.1 (-)
- new net Power Distribution/GND_BattboxFansL2: M3.1 (-), M4.1 (-)
- new net Power Distribution/GND_BattboxFansR1: M7.1 (-), M8.1 (-)
- new net Power Distribution/GND_BattboxFansR2: M10.1 (-), M9.1 (-)
- new net Power Distribution/IMD_Fault_Indicator: D102.2 (A)
- new net Power Distribution/IMD_Latch_Reset: SW107.1
- new net Power Distribution/SD_FromBrakeOT: SW101.2 (B)
- new net Power Distribution/SD_From_Side_BRBs: SW102.2 (B)
- new net Power Distribution/SD_ToBrakeOT: SW101.1 (A)
- new net Power Distribution/SD_ToCockpit: SW105.1 (A)
- new net Power Distribution/SD_To_Side_BRBs: SW103.2 (B)
- new net TSAL/GND: -108. (-)
- no-connect marks 13 -> 33
Other:
- removed sheet Segment 1
- removed sheet Segment 2
- removed sheet Segment 3
- removed sheet Segment 4
- removed sheet Segment 5
- removed sheet Segment 6
- added sheet Accumulator (Accumulator.kicad_sch)
- added sheet Accumulator Container (Accumulator_Container.kicad_sch)
- added sheet Brake_Light (Brake_Light.kicad_sch)
- added sheet Charger (Charger.kicad_sch)
- added sheet Charger1 (Charger.kicad_sch)
- added sheet Dashboard (Dashboard.kicad_sch)
- added sheet GLV Battery Board (GLV_Batt_Board.kicad_sch)
- added sheet LV_BOX (LV_BOX.kicad_sch)
- added sheet Mechanical_Sensor_Board_1 (MSB.kicad_sch)
- added sheet Mechanical_Sensor_Board_2 (MSB.kicad_sch)
- added sheet Mechanical_Sensor_Board_3 (MSB.kicad_sch)
- added sheet Power Distribution (PDU.kicad_sch)
- added sheet Steering_Wheel (Steering_Wheel.kicad_sch)
- added sheet TSAL (TSAL.kicad_sch)
- added sheet Wheel (Wheel.kicad_sch)
- note added: "(1) - When the charger GLV system is connected to the accumulator, power will be applied to the input of the GLVMS and power will drive the AIRs through the full shutdown loop"
- note added: "12AWG - Magenta2"
- note added: "14AWG"
- note added: "14AWG - Red3"
- note added: "16AWG"
- note added: "16AWG - Green3"
- note added: "17D Schematic for Reference"
- note added: "18AWG"
- note added: "18AWG - Yellow3"
- note added: "20AWG - Cyan3"
- note added: "22AWG"
- note added: "22AWG - Green Default(#009600FF)"
- note added: "26AWG - Orange1"
- note added: "2AWG - Orange3"
- note added: "30AWG - Magenta3"
- note added: "35 mm^2 - Orange4"
- note added: "35mm^2"
- note added: "3x 20AWG"
- note added: "8AWG"
- note added: "8AWG - Blue4"
- note added: "8x 22AWG"
- note added: "ACCUMULATOR COOLING"
- note added: "Accumulator"
- note added: "Accumulator Fans"
- note added: "All grounds marked with this symbol are directly grounded to the vehicle frame"
- note added: "BOLTED CONNECTION"
- note added: "Brake Light"
- note added: "Brake Pressure Sensors"
- note added: "CANBUS"
- note added: "Connected only while charging"
- note added: "Dashboard"
- note added: "Enclosed PCB containing relays and fuses for 12V power distribution. Also latching relays to open shutdown loop and latch in the event of faults"
- note added: "Fault Indicators located on the Dashboard"
- note added: "LFP Battery"
- note added: "MAIN TS"
- note added: "Motor Controller Shelf"
- note added: "Motor controller disconnected from TS while charging"
- note added: "NOTES"
- note added: "OFF VEHICLE"
- note added: "ON VEHICLE"
- note added: "Powertrain Cooling"
- note added: "Ready-to-Drive Sound"
- note added: "SHUTDOWN LOOP"
- note added: "TSMP and Shutdown Reset Container"
- note added: "Throttle Input"
- note added: "Wire Color Coding"
- note removed: "BMS"
- note removed: "Charger Shutdown"
- note removed: "HV"
- note removed: "Negative Sidepod"
- note removed: "OFFBOARD"
- note removed: "ONBOARD"
- note removed: "Positive Sidepod"
- moved on the sheet: U?
