File: NER22A/Shutdown_22A/Shutdown_22A.kicad_sch (KiCad schematic)
At the start: 63 parts, among them J1 GND, J2 TS+, J3 TS-, J4 Main TS Connector, K1 3PoleSwitchingRelay, K2 3PoleSwitchingRelay, K3 Omron DPDT Relay, K4 SPST-NO (Precharge Control), K5 SPST-NO (AIR Control), K6 SPST-NC (Discharge)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

Commit message: Fixed HV stuff
Parts:
- removed K4: SPST-NO (Precharge Control), Relay_THT:Relay_StandexMeder_DIP_LowProfile, symbol Relay:DIPxx-1Axx-11x
- removed R3: 5k, symbol Device:R
- removed SW9: HVD, symbol Switch:SW_SPST
- added K6: SPST-NC (Discharge), Relay_THT:Relay_SPST_StandexMeder_MS_Form1AB, symbol Relay:MSxx-1Bxx-75
- added K8 (x2): SPST-NO (AIR), Relay_THT:Relay_StandexMeder_DIP_LowProfile, symbol Relay:DIPxx-1Axx-11x
- added R4 (x2): 3.9k, symbol Device:R
- added SW7: HVD, symbol Switch:SW_SPST
- R4: value 1k -> 4.7k
Connections:
- net CHASSIS_GND: now also K6.5, K6.3, K8.2, K8.6; no longer K6.3
- net at F4.1, J4.1, K9.7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: now also K6.7
- net at F3.2, K6.1, K8.7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: now also SW7.2 (B); no longer J4.2
- net at K5.7, K5.8, K9.6: now also K6.3, K7.6, K6.5, K8.2, K8.6; no longer K6.5
- net at K6.7: now also R4.2
- net at BT4.1 (+): now also K8.7, K8.8
- net at BT3.2 (-): now also K8.1, K8.14
- net MotorController_AIRControl: no longer names the net of K5.6
- new net: K8.1, K8.14, K8.7, K8.8, R4.1, R4.2
- new net: J4.2, SW7.1 (A)
- new net: K6.1, R4.1
Other:
- note added: "PC Delay"
- moved on the sheet: BT4, BT5, J4, K5, K6, K9
